Commit message: update

File: src/Muuv_sim/muuv_sim_description/urdf/actuators.xacro (robot description, xacro)
@@ -1,6 +1,6 @@
 <?xml version="1.0"?>
 <robot xmlns:xacro="http://www.ros.org/wiki/xacro">
-    <!-- Adding the thruster units with the macro created in snippets.xacro -->
-    <!--
+  <!-- Adding the thruster units with the macro created in snippets.xacro -->
+  <!--
     Important:
         - The thruster IDs must be given as integers and must be unique to each thruster unit
@@ -8,15 +8,15 @@
           aware that Gazebo does not use the SNAME convention per default.
     -->
-    <xacro:thruster_macro robot_namespace="${namespace}" thruster_id="0">
-        <origin xyz="0 0 0" rpy="0 0 ${pi}" />
-    </xacro:thruster_macro>
-    <xacro:thruster_macro robot_namespace="${namespace}" thruster_id="1">
-        <origin xyz="0 0 0" rpy="0 0 ${pi}" />
-    </xacro:thruster_macro>
-    <xacro:thruster_macro robot_namespace="${namespace}" thruster_id="2">
-    <origin xyz="0 0 0" rpy="0 -${0.5*pi} 0" />
-    </xacro:thruster_macro>
-    <!-- Instantiate fins, if necessary -->
-    <!-- <xacro:fin_macro namespace="${namespace}" fin_id="0">
+  <xacro:T200_thruster_V2 robot_namespace="${namespace}" thruster_id="0">
+    <origin xyz="0 -0.470946 0.120758" rpy="-${0.5*pi} 0 0 " />
+  </xacro:T200_thruster_V2>
+  <xacro:T200_thruster_V2 robot_namespace="${namespace}" thruster_id="1">
+    <origin xyz="-0.10458 -0.470946 -0.060379" rpy="-${0.5*pi} 0 0" />
+  </xacro:T200_thruster_V2>
+  <xacro:T200_thruster_V2 robot_namespace="${namespace}" thruster_id="2">
+    <origin xyz="0.10458 -0.470946 -0.060379" rpy="-${0.5*pi} 0 0" />
+  </xacro:T200_thruster_V2>
+  <!-- Instantiate fins, if necessary -->
+  <!-- <xacro:fin_macro namespace="${namespace}" fin_id="0">
       <origin xyz="0 0 0" rpy="0 0 0" />
     </xacro:fin_macro>

File: src/Muuv_sim/muuv_sim_description/urdf/base.xacro (robot description, xacro)
@@ -8,11 +8,13 @@
   <xacro:include filename="$(find uuv_gazebo_ros_plugins)/urdf/snippets.xacro"/>
   <!-- Loading vehicle's specific macros -->
-  <xacro:include filename="$(find $CATKIN_PACKAGE)/urdf/snippets.xacro"/>
+  <!-- <xacro:include filename="$(find muuv_sim_description)/urdf/snippets.xacro"/> -->
+  <xacro:include filename="$(find muuv_sim_description)/urdf/thruster_types.xacro"/>
+  <xacro:include filename="$(find muuv_sim_description)/urdf/inertial_macros.xacro"/>
   <!--
     Vehicle's parameters (remember to enter the model parameters below)
   -->
-  <xacro:property name="mass" value="0"/>
+  <xacro:property name="mass" value="15"/>
   <!-- Center of gravity -->
-  <xacro:property name="cog" value="0 0 0"/>
+  <xacro:property name="cog" value="0 0 -0.08"/>
   <!-- Fluid density -->
   <xacro:property name="rho" value="1028"/>
@@ -23,37 +25,35 @@
     Open the meshes for the RexROV vehicle in Blender to see an example on the mesh placement.
   -->
-  <xacro:property name="visual_mesh_file" value="file://$(find $CATKIN_PACKAGE)/meshes/vehicle.dae"/>
+  <xacro:property name="visual_mesh_file" value="file://$(find muuv_sim_description)/meshes/vehicle.dae"/>
   <!-- Collision geometry mesh, usually in STL format (it is recommended to keep
   this geometry as simple as possible to improve the performance the physics engine
   regarding the computation of collision forces) -->
-  <xacro:property name="collision_mesh_file" value="file://$(find $CATKIN_PACKAGE)/meshes/vehicle.stl"/>
+  <xacro:property name="collision_mesh_file" value="file://$(find muuv_sim_description)/meshes/vehicle.stl"/>
   <!-- Vehicle macro -->
   <xacro:macro name="muuv_sim_base" params="namespace *gazebo">
-      <!-- Rigid body description of the base link -->
-      <link name="${namespace}/base_link">
-        <!--
+    <!-- Rigid body description of the base link -->
+    <link name="${namespace}/base_link">
+      <!--
           Be careful to setup the coefficients for the inertial tensor,
           otherwise your model will become unstable on Gazebo
         -->
-        <inertial>
-          <mass value="${mass}" />
-          <origin xyz="${cog}" rpy="0 0 0"/>
-          <inertia ixx="0" ixy="0" ixz="0"
-                   iyy="0" iyz="0"
-                   izz="0" />
-        </inertial>
-        <visual>
-          <origin xyz="0 0 0" rpy="0 0 0"/>
-          <geometry>
-            <mesh filename="${visual_mesh_file}" scale="1 1 1" />
-          </geometry>
-        </visual>
-        <collision>
-          <origin xyz="0 0 0" rpy="0 0 0"/>
-          <geometry>
-            <mesh filename="${collision_mesh_file}" scale="1 1 1" />
-          </geometry>
-        </collision>
-      </link>
+      <inertial>
+        <mass value="${mass}" />
+        <origin xyz="${cog}" rpy="0 0 0"/>
+        <inertia ixx="2.508" ixy="0" ixz="0" iyy="2.508" iyz="0" izz="0.10584"/>
+      </inertial>
+      <visual>
+        <origin xyz="0 0 0" rpy="0 0 0"/>
+        <geometry>
+          <mesh filename="${visual_mesh_file}" scale="1 1 1" />
+        </geometry>
+      </visual>
+      <collision>
+        <origin xyz="0 0 0" rpy="0 0 0"/>
+        <geometry>
+          <mesh filename="${collision_mesh_file}" scale="1 1 1" />
+        </geometry>
+      </collision>
+    </link>
     <gazebo reference="${namespace}/base_link">
       <selfCollide>false</selfCollide>
@@ -62,7 +62,7 @@
     <xacro:insert_block name="gazebo"/>
     <!-- Include the thruster modules -->
-    <xacro:include filename="$(find $CATKIN_PACKAGE)/urdf/actuators.xacro"/>
+    <xacro:include filename="$(find muuv_sim_description)/urdf/actuators.xacro"/>
     <!-- Include the sensor modules -->
-    <xacro:include filename="$(find $CATKIN_PACKAGE)/urdf/sensors.xacro"/>
+    <xacro:include filename="$(find muuv_sim_description)/urdf/sensors.xacro"/>
   </xacro:macro>
 </robot>

File: src/Muuv_sim/muuv_sim_description/urdf/gazebo.xacro (robot description, xacro)
@@ -2,11 +2,11 @@
 <robot xmlns:xacro="http://www.ros.org/wiki/xacro">
     <!-- Center of buoyancy -->
-    <xacro:property name="muuv_sim_cob" value="0 0 0"/>
+    <xacro:property name="muuv_sim_cob" value="0 0 0.08"/>
     <!-- Vehicle actual volume (Gazebo cannot compute the volume out of the mesh) -->
-    <xacro:property name="muuv_sim_volume" value="0"/>
+    <xacro:property name="muuv_sim_volume" value="0.024"/>
     <!-- Describing the dimensions of the vehicle bounding box -->
-    <xacro:property name="muuv_sim_length" value="0"/>
-    <xacro:property name="muuv_sim_width"  value="0"/>
-    <xacro:property name="muuv_sim_height" value="0"/>
+    <xacro:property name="muuv_sim_length" value="0.146"/>
+    <xacro:property name="muuv_sim_width"  value="0.991"/>
+    <xacro:property name="muuv_sim_height" value="0.168"/>
     <xacro:macro name="muuv_sim_hydro_model" params="namespace">
       <!-- List of hydrodynamic models this robot links -->
@@ -50,5 +50,5 @@
           <linear_damping>
             0 0 0 0 0 0
-          </linear_damping>
+        </linear_damping>
           <!--
             The linear damping coefficients proportional to the forward speed
@@ -66,5 +66,5 @@
           <quadratic_damping>
             0 0 0 0 0 0
-          </quadratic_damping>
+        </quadratic_damping>
           <!--
             In case you want to model a simple surface vessel, you can use the
@@ -91,5 +91,5 @@
         <hydrodynamic_model>
           <type>sphere</type>
-          <radius>0</radius>
+          <radius>1</radius>
         </hydrodynamic_model>
       </link>

File: src/Muuv_sim/muuv_sim_description/urdf/sensors.xacro (robot description, xacro)
@@ -12,15 +12,15 @@
   <xacro:default_pose_3d namespace="${namespace}" parent_link="${namespace}/base_link" />
   <!-- Forward-looking sonar sensor -->
-  <!-- <xacro:forward_multibeam_p900 namespace="${namespace}" parent_link="${namespace}/base_link"> -->
-    <!-- <origin xyz="0 0 0" rpy="0 0 0"/> -->
-  <!-- </xacro:forward_multibeam_p900> -->
+  <!-- <xacro:forward_multibeam_p900 namespace="${namespace}" parent_link="${namespace}/base_link">
+    <origin xyz="0 0 0" rpy="0 0 0"/>
+  </xacro:forward_multibeam_p900> -->
   <!-- DVL  -->
-  <!-- <xacro:default_dvl namespace="${namespace}" parent_link="${namespace}/base_link"> -->
-    <!-- <origin xyz="0 0 0" rpy="0 0 0"/> -->
-  <!-- </xacro:default_dvl> -->
+  <!-- <xacro:default_dvl namespace="${namespace}" parent_link="${namespace}/base_link">
+    <origin xyz="0 0 0" rpy="0 0 0"/>
+  </xacro:default_dvl> -->
   <!-- RPT  -->
-  <!-- <xacro:default_rpt namespace="${namespace}" parent_link="${namespace}/base_link"> -->
-    <!-- <origin xyz="0 0 0" rpy="0 0 0"/> -->
-  <!-- </xacro:default_rpt> -->
+  <!-- <xacro:default_rpt namespace="${namespace}" parent_link="${namespace}/base_link">
+    <origin xyz="0 0 0" rpy="0 0 0"/>
+  </xacro:default_rpt> -->
   <!-- Pressure  -->
   <xacro:default_pressure namespace="${namespace}" parent_link="${namespace}/base_link">
@@ -32,6 +32,6 @@
   </xacro:default_imu>
   <!-- Mount a camera  -->
-  <!-- <xacro:default_camera namespace="${namespace}" parent_link="${namespace}/base_link" suffix=""> -->
-    <!-- <origin xyz="0 0 0" rpy="0 0 0"/>
-  </xacro:default_camera> -->
+  <xacro:default_camera namespace="${namespace}" parent_link="${namespace}/base_link" suffix="">
+    <origin xyz="0 0.6 0" rpy="0 0 0"/>
+  </xacro:default_camera>
 </robot>

File: src/Muuv_sim/muuv_sim_description/urdf/snippets.xacro (robot description, xacro)
@@ -7,5 +7,5 @@
   over propeller's frame X-axis in DAE (Collada) or STL format.
   -->
-  <xacro:property name="prop_mesh_file" value="file://$(find $CATKIN_PACKAGE)/meshes/propeller.dae"/>
+  <xacro:property name="prop_mesh_file" value="file://$(find muuv_sim_description)/meshes/T200_Thruster.dae"/>
   <!--
     Thruster macro with integration of joint and link. The thrusters should
@@ -164,5 +164,5 @@
   -->
   <!-- A separate mesh for the fin should be stored in the meshes folder -->
-  <xacro:property name="fin_mesh_file" value="file://$(find $CATKIN_PACKAGE)/meshes/fin.dae"/>
+  <xacro:property name="fin_mesh_file" value="file://$(find muuv_sim_description)/meshes/fin.dae"/>
   <!-- Fin joint limits  -->
   <xacro:property name="fin_min_joint_limit" value="${0.0 * d2r}"/>
